File: arduino_isp_pcb/arduino_isp_pcb.sch (KiCad schematic (older format))
At the start: 8 parts, among them J1 Conn_02x05_Odd_Even

Commit message: PCB: add pcb
Route PCB
Parts:
- R1, R2, R3: footprint Resistor_THT:R_Axial_DIN0309_L9.0mm_D3.2mm_P12.70mm_Horizontal -> Resistor_SMD:R_0805_2012Metric_Pad1.15x1.40mm_HandSolder
Changed lines of the file:
@@
 F 0 "R1" V 7543 4450 50  0000 C CNN
 F 1 "R" V 7634 4450 50  0000 C CNN
-F 2 "Resistor_THT:R_Axial_DIN0309_L9.0mm_D3.2mm_P12.70mm_Horizontal" V 7680 4450 50  0001 C CNN
+F 2 "Resistor_SMD:R_0805_2012Metric_Pad1.15x1.40mm_HandSolder" V 7680 4450 50  0001 C CNN
 F 3 "~" H 7750 4450 50  0001 C CNN
 	1    7750 4450
@@
 F 0 "R2" V 7543 4900 50  0000 C CNN
 F 1 "R" V 7634 4900 50  0000 C CNN
-F 2 "Resistor_THT:R_Axial_DIN0309_L9.0mm_D3.2mm_P12.70mm_Horizontal" V 7680 4900 50  0001 C CNN
+F 2 "Resistor_SMD:R_0805_2012Metric_Pad1.15x1.40mm_HandSolder" V 7680 4900 50  0001 C CNN
 F 3 "~" H 7750 4900 50  0001 C CNN
 	1    7750 4900
@@
 F 0 "R3" V 7543 5350 50  0000 C CNN
 F 1 "R" V 7634 5350 50  0000 C CNN
-F 2 "Resistor_THT:R_Axial_DIN0309_L9.0mm_D3.2mm_P12.70mm_Horizontal" V 7680 5350 50  0001 C CNN
+F 2 "Resistor_SMD:R_0805_2012Metric_Pad1.15x1.40mm_HandSolder" V 7680 5350 50  0001 C CNN
 F 3 "~" H 7750 5350 50  0001 C CNN
 	1    7750 5350

Commit message: PCB: add 6 pins AVR ISP connector
Parts:
- added J2: Conn_02x03_Odd_Even, Connector_PinHeader_2.54mm:PinHeader_2x03_P2.54mm_Vertical, symbol Connector_Generic:Conn_02x03_Odd_Even
- J1: footprint Connector_PinSocket_2.54mm:PinSocket_2x05_P2.54mm_Vertical -> Connector_PinHeader_2.54mm:PinHeader_2x05_P2.54mm_Vertical
Connections:
- wire segments 36 -> 42
Changed lines of the file:
@@
 F 0 "J1" H 8000 3717 50  0000 C CNN
 F 1 "Conn_02x05_Odd_Even" H 8000 3626 50  0000 C CNN
-F 2 "Connector_PinSocket_2.54mm:PinSocket_2x05_P2.54mm_Vertical" H 7950 3300 50  0001 C CNN
+F 2 "Connector_PinHeader_2.54mm:PinHeader_2x05_P2.54mm_Vertical" H 7950 3300 50  0001 C CNN
 F 3 "~" H 7950 3300 50  0001 C CNN
 	1    7950 3300
@@
 Wire Wire Line
 	8600 5350 8600 5450
+$Comp
+L Connector_Generic:Conn_02x03_Odd_Even J2
+U 1 1 5B5EFDA9
+P 7900 1350
+F 0 "J2" H 7950 1667 50  0000 C CNN
+F 1 "Conn_02x03_Odd_Even" H 7950 1576 50  0000 C CNN
+F 2 "Connector_PinHeader_2.54mm:PinHeader_2x03_P2.54mm_Vertical" H 7900 1350 50  0001 C CNN
+F 3 "~" H 7900 1350 50  0001 C CNN
+	1    7900 1350
+	1    0    0    -1
+$EndComp
+$Comp
+L power:GND #PWR06
+U 1 1 5B5EFF13
+P 8300 1450
+F 0 "#PWR06" H 8300 1200 50  0001 C CNN
+F 1 "GND" H 8305 1277 50  0000 C CNN
+F 2 "" H 8300 1450 50  0001 C CNN
+F 3 "" H 8300 1450 50  0001 C CNN
+	1    8300 1450
+	1    0    0    -1
+$EndComp
+$Comp
+L power:+5V #PWR07
+U 1 1 5B5EFF30
+P 8500 1250
+F 0 "#PWR07" H 8500 1100 50  0001 C CNN
+F 1 "+5V" H 8515 1423 50  0000 C CNN
+F 2 "" H 8500 1250 50  0001 C CNN
+F 3 "" H 8500 1250 50  0001 C CNN
+	1    8500 1250
+	1    0    0    -1
+$EndComp
+Wire Wire Line
+	8200 1250 8500 1250
+Wire Wire Line
+	8300 1450 8200 1450
+Text GLabel 8450 1350 2    50   Input ~ 0
+MOSI
+Text GLabel 7400 1250 0    50   Input ~ 0
+MISO
+Text GLabel 7400 1350 0    50   Input ~ 0
+SCLK
+Text GLabel 7400 1450 0    50   Input ~ 0
+T_RST
+Wire Wire Line
+	7400 1450 7700 1450
+Wire Wire Line
+	7400 1350 7700 1350
+Wire Wire Line
+	7400 1250 7700 1250
+Wire Wire Line
+	8200 1350 8450 1350
 $EndSCHEMATC
